File: CubeSat-Comms-XCVR-PCB-Fall2025-Version.kicad_pcb (KiCad board)
At the start: 4 copper layers, 100 x 100 mm, 68 parts, among them J1 Screw_Terminal_01x02, J2 Screw_Terminal_01x02, J3 Conn_Coaxial, J4 Conn_01x12_Pin, U1 CC1101RGP, U2 SKY65366-21, U3 PE4251MLI-Z, U4 NCP186AMX390TAG, Y1 NX3225GA-26MHZ-TI

Commit message: Update KiCad project
Parts:
- moved H3 10.6 mm to (111.7, 140.6)
- moved H4 8.03 mm to (191.4, 140.6)
- moved H1 4.79 mm to (195.3, 52.2)
- moved H2 2.32 mm to (109.1, 52.2)
Changed lines of the file:
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@@
 	(footprint "MountingHole:MountingHole_2.2mm_M2"
 		(layer "F.Cu")
-		(at 199.345301 49.7207)
+		(at 195.252301 52.2119)
 		(descr "Mounting Hole 2.2mm, M2, no annular, generated by kicad-footprint-generator mountinghole.py")
 		(tags "mountinghole M2")
@@
 	(footprint "MountingHole:MountingHole_2.2mm_M2"
 		(layer "F.Cu")
-		(at 102.745301 146.4207)
+		(at 111.660701 140.6295)
 		(descr "Mounting Hole 2.2mm, M2, no annular, generated by kicad-footprint-generator mountinghole.py")
 		(tags "mountinghole M2")
@@
 	(footprint "MountingHole:MountingHole_2.2mm_M2"
 		(layer "F.Cu")
-		(at 107.345301 50.7207)
+		(at 109.120701 52.2119)
 		(descr "Mounting Hole 2.2mm, M2, no annular, generated by kicad-footprint-generator mountinghole.py")
 		(tags "mountinghole M2")
@@
 	(footprint "MountingHole:MountingHole_2.2mm_M2"
 		(layer "F.Cu")
-		(at 199.045301 143.2207)
+		(at 191.442301 140.6295)
 		(descr "Mounting Hole 2.2mm, M2, no annular, generated by kicad-footprint-generator mountinghole.py")
 		(tags "mountinghole M2")

Commit message: Update KiCad project
Parts:
- moved J1 88.1 mm to (177.5, 140.5), turned to 180 degrees
- moved D1 76.8 mm to (174.5, 134.9), turned to 180 degrees
- moved D3 73.1 mm to (177.9, 132.9), turned to 180 degrees
- moved R2 72.8 mm to (173.9, 132.9), turned to 0 degrees
- moved D2 54.1 mm to (191.0, 125.1)
- moved J2 54.1 mm to (197.1, 122.8)
- moved R3 54.1 mm to (189.5, 127.2)
- moved D4 54.1 mm to (189.5, 123.2)
- moved J3 53.5 mm to (193.0, 100.0), turned to 180 degrees
- moved C29 44.6 mm to (187.0, 97.9), turned to 90 degrees
- moved L5 44.1 mm to (184.8, 100.7), turned to 180 degrees
- moved C31 42.0 mm to (184.5, 98.5), turned to 180 degrees
- moved R4 41.6 mm to (181.9, 103.1), turned to 180 degrees
- moved C30 39.3 mm to (181.7, 99.1), turned to -90 degrees
- moved C28 35.8 mm to (179.1, 101.1)
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Routing:
- net VPC: track 33.3 -> 81.3 mm
- net BYP: track 38.7 -> 81.0 mm
- net EN: track 39.4 -> 80.3 mm
- net TR: track 39.3 -> 79.4 mm
- net +3.9V: track 37.5 -> 13.3 mm, vias 2 -> 0
- net CSN: track 44.6 -> 22.7 mm, vias 2 -> 0
- net Net-(J3-Ext): track 8.09 -> 28.4 mm
- net GD02: track 39.5 -> 22.4 mm
- net GND: track 144.9 -> 128.9 mm, vias 23 -> 24
- net +3.3V: track 94.2 -> 79.0 mm
- net RF1_STATUS: track 80.0 -> 94.3 mm
- net SO: track 37.1 -> 22.9 mm
- net SCLK: track 37.1 -> 24.0 mm
- net RFC: track 17.2 -> 5.72 mm
- net GD00: track 40.1 -> 29.2 mm
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Other:
- outline, holes or cut-outs redrawn
- board text added: "+3.3V"
- board text added: "+5V"
- board text added: "Ant"
- board text added: "LNA Network"
- board text added: "PA Network"
- board text added: "RF Switch"
- board text added: "SAW Filter"
- board text added: "STM32 ControlS"
- board text added: "Transceiver"
- board text added: "XCVR_CLK"
