File: CubeSat-Comms-XCVR-PCB-Fall2025-Version.kicad_sch (KiCad schematic)
At the start: 81 parts, among them J1 Conn_01x02_Pin, J10 Conn_Coaxial, J12 Conn_01x04_Pin, J2 Conn_01x02_Pin, J3 Conn_Coaxial, J4 Conn_01x12_Pin, J5 Conn_01x02_Pin, J6 Conn_01x02_Pin, J7 Conn_01x02_Pin, J8 Conn_01x02_Pin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

Commit message: empty commit
Connections:
- net GND: now also U4.3 (N/C)
Other:
- moved on the sheet: C21, D5, R6
